File: hardware/pn_ecp5_evn/pn_wing_prototype.kicad_pcb (KiCad board)
At the start: 4 copper layers, 129.5 x 52.2 mm, 277 parts, among them J101 Screw_Terminal_01x02, J102 Conn_Coaxial, J103 Conn_02x20_Odd_Even, J104 Conn_Coaxial, J105 Conn_Coaxial, J106 Conn_Coaxial, J107 Conn_01x10, J201 Conn_Coaxial, J301 Conn_Coaxial, J401 Conn_Coaxial, J601 Conn_Coaxial, J701 Conn_Coaxial, J702 Conn_Coaxial, J703 Conn_Coaxial, U201 VEMI65AB-HCI, U202 LMX2594, U301 PAT1220-C-3DB, U302 TRF37A73, U303 PAT1220-C-3DB, U401 PAT1220-C-3DB, U402 TRF37A73, U403 PAT1220-C-3DB, U501 LM27761, U502 ADM7171ACPZ-3.3-R7, U503 TPS72301DB, U601 LM2904, U602 OPA2211, U701 SYM-63LH+, U702 ADG621, U703 OPA2211, U801 THS4551, U802 LT6657BHMS8-2.5, U901 ADS7868, U902 ADS7868, U903 Si8640BB-B-IU, U904 Si8640BB-B-IU, U905 Si8642BB-B-IU, X601 ABLNO

Commit message: added assembly drawing
Parts:
- C805: value 470 pF -> DNI
- C806: value 1 nF -> DNI
- C810, C811: value 270 pF -> DNI
- R207: value 0k -> 18
- R803: value 1.2k -> 187
- R804: value 1.2k -> 215
- R805, R806: value 330 -> 0
- R808, R811: value 1.2k -> DNI
- R809, R810: value DNI -> 1k
- R818: value 1.2k -> 51
- R819: value 1.2k -> 59
- U802: value LT6657BHMS8-2.5 -> DNI
Changed lines of the file:
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@@
   )
   (setup
-    (last_trace_width 0.32)
+    (last_trace_width 0.25)
     (user_trace_width 0.13)
     (user_trace_width 0.2)
@@
       (effects (font (size 1 1) (thickness 0.15)))
     )
-    (fp_text user %R (at 0 0) (layer F.Fab)
-      (effects (font (size 0.25 0.25) (thickness 0.04)))
-    )
     (fp_line (start -0.5 0.25) (end -0.5 -0.25) (layer F.Fab) (width 0.1))
     (fp_line (start -0.5 -0.25) (end 0.5 -0.25) (layer F.Fab) (width 0.1))
@@
     (fp_line (start 0.93 -0.47) (end 0.93 0.47) (layer F.CrtYd) (width 0.05))
     (fp_line (start 0.93 0.47) (end -0.93 0.47) (layer F.CrtYd) (width 0.05))
+    (fp_text user %R (at 0 0) (layer F.Fab)
+      (effects (font (size 0.25 0.25) (thickness 0.04)))
+    )
     (pad 2 smd roundrect (at 0.485 0 180) (size 0.59 0.64) (layers F.Cu F.Paste F.Mask) (roundrect_rratio 0.25)
       (net 192 "Net-(C813-Pad2)"))
@@
       (effects (font (size 1 1) (thickness 0.15)))
     )
-    (fp_text user %R (at 0 0) (layer F.Fab)
-      (effects (font (size 0.25 0.25) (thickness 0.04)))
-    )
     (fp_line (start -0.5 0.25) (end -0.5 -0.25) (layer F.Fab) (width 0.1))
     (fp_line (start -0.5 -0.25) (end 0.5 -0.25) (layer F.Fab) (width 0.1))
@@
     (fp_line (start 0.93 -0.47) (end 0.93 0.47) (layer F.CrtYd) (width 0.05))
     (fp_line (start 0.93 0.47) (end -0.93 0.47) (layer F.CrtYd) (width 0.05))
+    (fp_text user %R (at 0 0) (layer F.Fab)
+      (effects (font (size 0.25 0.25) (thickness 0.04)))
+    )
     (pad 2 smd roundrect (at 0.485 0) (size 0.59 0.64) (layers F.Cu F.Paste F.Mask) (roundrect_rratio 0.25)
       (net 191 "Net-(C813-Pad1)"))
@@
       (effects (font (size 1 1) (thickness 0.15)))
     )
-    (fp_text user %R (at 0 0) (layer F.Fab)
-      (effects (font (size 0.25 0.25) (thickness 0.04)))
-    )
     (fp_line (start -0.5 0.25) (end -0.5 -0.25) (layer F.Fab) (width 0.1))
     (fp_line (start -0.5 -0.25) (end 0.5 -0.25) (layer F.Fab) (width 0.1))
@@
     (fp_line (start 0.93 -0.47) (end 0.93 0.47) (layer F.CrtYd) (width 0.05))
     (fp_line (start 0.93 0.47) (end -0.93 0.47) (layer F.CrtYd) (width 0.05))
+    (fp_text user %R (at 0 0) (layer F.Fab)
+      (effects (font (size 0.25 0.25) (thickness 0.04)))
+    )
     (pad 2 smd roundrect (at 0.485 0 180) (size 0.59 0.64) (layers F.Cu F.Paste F.Mask) (roundrect_rratio 0.25)
       (net 191 "Net-(C813-Pad1)"))
@@
       (effects (font (size 0.7 0.7) (thickness 0.15)))
     )
-    (fp_text value 1.2k (at 0 1.17 90) (layer F.Fab)
+    (fp_text value 59 (at 0 1.17 90) (layer F.Fab)
       (effects (font (size 1 1) (thickness 0.15)))
     )
-    (fp_text user %R (at 0 0 90) (layer F.Fab)
-      (effects (font (size 0.25 0.25) (thickness 0.04)))
-    )
     (fp_line (start -0.5 0.25) (end -0.5 -0.25) (layer F.Fab) (width 0.1))
     (fp_line (start -0.5 -0.25) (end 0.5 -0.25) (layer F.Fab) (width 0.1))
@@
     (fp_line (start 0.93 -0.47) (end 0.93 0.47) (layer F.CrtYd) (width 0.05))
     (fp_line (start 0.93 0.47) (end -0.93 0.47) (layer F.CrtYd) (width 0.05))
+    (fp_text user %R (at 0 0 90) (layer F.Fab)
+      (effects (font (size 0.25 0.25) (thickness 0.04)))
+    )
     (pad 2 smd roundrect (at 0.485 0 270) (size 0.59 0.64) (layers F.Cu F.Paste F.Mask) (roundrect_rratio 0.25)
       (net 1 GND))
@@
       (effects (font (size 0.7 0.7) (thickness 0.15)))
     )
-    (fp_text value 1.2k (at 0 1.17 90) (layer F.Fab)
+    (fp_text value 51 (at 0 1.17 90) (layer F.Fab)
       (effects (font (size 1 1) (thickness 0.15)))
     )
-    (fp_text user %R (at 0 0 90) (layer F.Fab)
-      (effects (font (size 0.25 0.25) (thickness 0.04)))
-    )
     (fp_line (start -0.5 0.25) (end -0.5 -0.25) (layer F.Fab) (width 0.1))
     (fp_line (start -0.5 -0.25) (end 0.5 -0.25) (layer F.Fab) (width 0.1))
@@
     (fp_line (start 0.93 -0.47) (end 0.93 0.47) (layer F.CrtYd) (width 0.05))
     (fp_line (start 0.93 0.47) (end -0.93 0.47) (layer F.CrtYd) (width 0.05))
+    (fp_text user %R (at 0 0 90) (layer F.Fab)
+      (effects (font (size 0.25 0.25) (thickness 0.04)))
+    )
     (pad 2 smd roundrect (at 0.485 0 270) (size 0.59 0.64) (layers F.Cu F.Paste F.Mask) (roundrect_rratio 0.25)
       (net 141 /adc/ADC_VIN))
@@
       (effects (font (size 1 1) (thickness 0.15)))
     )
-    (fp_text user %R (at 0 0 90) (layer F.Fab)
-      (effects (font (size 0.4 0.4) (thickness 0.06)))
-    )
     (fp_line (start -0.8 0.4) (end -0.8 -0.4) (layer F.Fab) (width 0.1))
     (fp_line (start -0.8 -0.4) (end 0.8 -0.4) (layer F.Fab) (width 0.1))
@@
     (fp_line (start 1.48 -0.73) (end 1.48 0.73) (layer F.CrtYd) (width 0.05))
     (fp_line (start 1.48 0.73) (end -1.48 0.73) (layer F.CrtYd) (width 0.05))
+    (fp_text user %R (at 0 0 90) (layer F.Fab)
+      (effects (font (size 0.4 0.4) (thickness 0.06)))
+    )
     (pad 2 smd roundrect (at 0.7875 0 90) (size 0.875 0.95) (layers F.Cu F.Paste F.Mask) (roundrect_rratio 0.25)
       (net 192 "Net-(C813-Pad2)"))
@@
       (effects (font (size 1 1) (thickness 0.15)))
     )
-    (fp_text user %R (at 0 0 90) (layer F.Fab)
-      (effects (font (size 0.4 0.4) (thickness 0.06)))
-    )
     (fp_line (start -0.8 0.4) (end -0.8 -0.4) (layer F.Fab) (width 0.1))
     (fp_line (start -0.8 -0.4) (end 0.8 -0.4) (layer F.Fab) (width 0.1))
@@
     (fp_line (start 1.48 -0.73) (end 1.48 0.73) (layer F.CrtYd) (width 0.05))
     (fp_line (start 1.48 0.73) (end -1.48 0.73) (layer F.CrtYd) (width 0.05))
+    (fp_text user %R (at 0 0 90) (layer F.Fab)
+      (effects (font (size 0.4 0.4) (thickness 0.06)))
+    )
     (pad 2 smd roundrect (at 0.7875 0 90) (size 0.875 0.95) (layers F.Cu F.Paste F.Mask) (roundrect_rratio 0.25)
       (net 191 "Net-(C813-Pad1)"))
@@
       (effects (font (size 0.7 0.7) (thickness 0.15)))
     )
-    (fp_text value "270 pF" (at 0 1.43 90) (layer F.Fab)
+    (fp_text value DNI (at 0 1.43 90) (layer F.Fab)
       (effects (font (size 1 1) (thickness 0.15)))
     )
@@
       (effects (font (size 0.7 0.7) (thickness 0.15)))
     )
-    (fp_text value "270 pF" (at 0 1.43 90) (layer F.Fab)
+    (fp_text value DNI (at 0 1.43 90) (layer F.Fab)
       (effects (font (size 1 1) (thickness 0.15)))
     )
@@
       (effects (font (size 0.7 0.7) (thickness 0.15)))
     )
-    (fp_text value "470 pF" (at 0 1.43 90) (layer F.Fab)
+    (fp_text value DNI (at 0 1.43 90) (layer F.Fab)
       (effects (font (size 1 1) (thickness 0.15)))
     )
@@
       (effects (font (size 0.7 0.7) (thickness 0.15)))
     )
-    (fp_text value LT6657BHMS8-2.5 (at 0 2.45 90) (layer F.Fab)
+    (fp_text value DNI (at 0 2.45 90) (layer F.Fab)
       (effects (font (size 1 1) (thickness 0.15)))
     )
@@
       (effects (font (size 0.7 0.7) (thickness 0.15)))
     )
-    (fp_text value 1.2k (at 0 1.17 90) (layer F.Fab)
+    (fp_text value DNI (at 0 1.17 90) (layer F.Fab)
       (effects (font (size 1 1) (thickness 0.15)))
     )
@@
       (effects (font (size 0.7 0.7) (thickness 0.15)))
     )
-    (fp_text value DNI (at 0 1.17 90) (layer F.Fab)
+    (fp_text value 1k (at 0 1.17 90) (layer F.Fab)
       (effects (font (size 1 1) (thickness 0.15)))
     )
@@
       (effects (font (size 0.7 0.7) (thickness 0.15)))
     )
-    (fp_text value DNI (at 0 1.17 90) (layer F.Fab)
+    (fp_text value 1k (at 0 1.17 90) (layer F.Fab)
       (effects (font (size 1 1) (thickness 0.15)))
     )
@@
       (effects (font (size 0.7 0.7) (thickness 0.15)))
     )
-    (fp_text value 1.2k (at 0 1.17 90) (layer F.Fab)
+    (fp_text value DNI (at 0 1.17 90) (layer F.Fab)
       (effects (font (size 1 1) (thickness 0.15)))
     )
@@
       (effects (font (size 0.7 0.7) (thickness 0.15)))
     )
-    (fp_text value 330 (at 0 1.17) (layer F.Fab)
+    (fp_text value 0 (at 0 1.17) (layer F.Fab)
       (effects (font (size 1 1) (thickness 0.15)))
     )
@@
       (effects (font (size 0.7 0.7) (thickness 0.15)))
     )
-    (fp_text value 330 (at 0 1.17) (layer F.Fab)
+    (fp_text value 0 (at 0 1.17) (layer F.Fab)
       (effects (font (size 1 1) (thickness 0.15)))
     )
@@
       (effects (font (size 0.7 0.7) (thickness 0.15)))
     )
-    (fp_text value 1.2k (at 0 1.17 90) (layer F.Fab)
+    (fp_text value 215 (at 0 1.17 90) (layer F.Fab)
       (effects (font (size 1 1) (thickness 0.15)))
     )
@@
       (effects (font (size 0.7 0.7) (thickness 0.15)))
     )
-    (fp_text value 1.2k (at 0 1.17 90) (layer F.Fab)
+    (fp_text value 187 (at 0 1.17 90) (layer F.Fab)
       (effects (font (size 1 1) (thickness 0.15)))
     )
@@
       (effects (font (size 0.7 0.7) (thickness 0.15)))
     )
-    (fp_text value 0k (at 0 1.17) (layer F.Fab)
+    (fp_text value 18 (at 0 1.17) (layer F.Fab)
       (effects (font (size 1 1) (thickness 0.15)))
     )
@@
       (effects (font (size 0.7 0.7) (thickness 0.15)))
     )
-    (fp_text value "1 nF" (at 0 1.17 90) (layer F.Fab)
+    (fp_text value DNI (at 0 1.17 90) (layer F.Fab)
       (effects (font (size 1 1) (thickness 0.15)))
     )
